File: Debugger-PCB/PowerAndPort.kicad_sch (KiCad schematic)
At the start: 22 parts, among them J1 Conn_01x04, J2 Conn_01x04, J3 Conn_01x02, J4 USB_C_Receptacle_USB2.0, U1 HX9193, U2 HX9193, U3 CH340E, U4 TJA1051T-3

Commit message: fix some details of PCB
Parts:
- added R10, R11: 10k, Resistor_SMD:R_0603_1608Metric, symbol Device:R_Small
Connections:
- net CAN+: now also R10.2
- net CAN-: now also R11.1
- net GND: now also R10.1, R11.2
Changed lines of the file:
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@@
   (junction (at 234.95 140.97) (diameter 0) (color 0 0 0 0)
   )
+  (junction (at 254 127) (diameter 0) (color 0 0 0 0)
+  )
   (junction (at 218.44 54.61) (diameter 0) (color 0 0 0 0)
   )
   (junction (at 226.06 48.26) (diameter 0) (color 0 0 0 0)
+  )
+  (junction (at 254 132.08) (diameter 0) (color 0 0 0 0)
   )
   (junction (at 67.31 132.08) (diameter 0) (color 0 0 0 0)
@@
     (stroke (width 0) (type default) (color 0 0 0 0))
   )
+  (wire (pts (xy 254 140.97) (xy 254 139.7))
+    (stroke (width 0) (type default) (color 0 0 0 0))
+  )
   (wire (pts (xy 152.4 98.298) (xy 152.4 99.06))
     (stroke (width 0) (type default) (color 0 0 0 0))
@@
     (stroke (width 0) (type default) (color 0 0 0 0))
   )
+  (wire (pts (xy 254 124.46) (xy 254 127))
+    (stroke (width 0) (type default) (color 0 0 0 0))
+  )
   (wire (pts (xy 74.93 52.07) (xy 68.58 52.07))
     (stroke (width 0) (type default) (color 0 0 0 0))
@@
     (stroke (width 0) (type default) (color 0 0 0 0))
   )
+  (wire (pts (xy 262.255 117.475) (xy 262.255 119.38))
+    (stroke (width 0) (type default) (color 0 0 0 0))
+  )
   (wire (pts (xy 218.44 48.26) (xy 226.06 48.26))
     (stroke (width 0) (type default) (color 0 0 0 0))
@@
     (stroke (width 0) (type default) (color 0 0 0 0))
   )
+  (wire (pts (xy 254 119.38) (xy 254 117.475))
+    (stroke (width 0) (type default) (color 0 0 0 0))
+  )
   (wire (pts (xy 152.4 99.06) (xy 152.4 100.33))
     (stroke (width 0) (type default) (color 0 0 0 0))
@@
     (stroke (width 0) (type default) (color 0 0 0 0))
   )
+  (wire (pts (xy 254 117.475) (xy 262.255 117.475))
+    (stroke (width 0) (type default) (color 0 0 0 0))
+  )
   (wire (pts (xy 67.31 132.08) (xy 67.31 132.842))
     (stroke (width 0) (type default) (color 0 0 0 0))
@@
   )
   (wire (pts (xy 73.66 54.61) (xy 74.93 54.61))
+    (stroke (width 0) (type default) (color 0 0 0 0))
+  )
+  (wire (pts (xy 254 132.08) (xy 254 134.62))
     (stroke (width 0) (type default) (color 0 0 0 0))
   )
@@
     (pin "1")
   )
+  (symbol (lib_id "Device:R_Small") (at 254 137.16 0) (unit 1)
+    (in_bom yes) (on_board yes)
+    (property "Reference" "R11" (id 0) (at 255.4986 136.2515 0)
+      (effects (font (size 1.27 1.27)) (justify left))
+    )
+    (property "Value" "10k" (id 1) (at 255.27 138.811 0)
+      (effects (font (size 1.27 1.27)) (justify left))
+    )
+    (property "Footprint" "Resistor_SMD:R_0603_1608Metric" (id 2) (at 254 137.16 0)
+      (effects (font (size 1.27 1.27)) hide)
+    )
+    (property "Datasheet" "~" (id 3) (at 254 137.16 0)
+      (effects (font (size 1.27 1.27)) hide)
+    )
+    (pin "1")
+    (pin "2")
+  )
   (symbol (lib_id "power:+5V") (at 234.95 116.84 0) (unit 1)
     (in_bom yes) (on_board yes) (fields_autoplaced)
@@
     (pin "4")
     (pin "5")
+  )
+  (symbol (lib_id "power:GND") (at 254 140.97 0) (unit 1)
+    (in_bom yes) (on_board yes) (fields_autoplaced)
+    (property "Reference" "#PWR0104" (id 0) (at 254 147.32 0)
+      (effects (font (size 1.27 1.27)) hide)
+    )
+    (property "Value" "GND" (id 1) (at 254 145.5325 0))
+    (property "Footprint" "" (id 2) (at 254 140.97 0)
+      (effects (font (size 1.27 1.27)) hide)
+    )
+    (property "Datasheet" "" (id 3) (at 254 140.97 0)
+      (effects (font (size 1.27 1.27)) hide)
+    )
+    (pin "1")
   )
   (symbol (lib_id "Connector:USB_C_Receptacle_USB2.0") (at 67.31 109.22 0) (unit 1)
@@
     (pin "1")
   )
+  (symbol (lib_id "Device:R_Small") (at 254 121.92 0) (unit 1)
+    (in_bom yes) (on_board yes)
+    (property "Reference" "R10" (id 0) (at 255.4986 121.0115 0)
+      (effects (font (size 1.27 1.27)) (justify left))
+    )
+    (property "Value" "10k" (id 1) (at 255.27 123.571 0)
+      (effects (font (size 1.27 1.27)) (justify left))
+    )
+    (property "Footprint" "Resistor_SMD:R_0603_1608Metric" (id 2) (at 254 121.92 0)
+      (effects (font (size 1.27 1.27)) hide)
+    )
+    (property "Datasheet" "~" (id 3) (at 254 121.92 0)
+      (effects (font (size 1.27 1.27)) hide)
+    )
+    (pin "1")
+    (pin "2")
+  )
   (symbol (lib_id "power:GND") (at 182.88 66.04 0) (unit 1)
     (in_bom yes) (on_board yes) (fields_autoplaced)
@@
     (pin "2")
   )
+  (symbol (lib_id "power:GND") (at 262.255 119.38 0) (unit 1)
+    (in_bom yes) (on_board yes) (fields_autoplaced)
+    (property "Reference" "#PWR0105" (id 0) (at 262.255 125.73 0)
+      (effects (font (size 1.27 1.27)) hide)
+    )
+    (property "Value" "GND" (id 1) (at 262.255 123.9425 0))
+    (property "Footprint" "" (id 2) (at 262.255 119.38 0)
+      (effects (font (size 1.27 1.27)) hide)
+    )
+    (property "Datasheet" "" (id 3) (at 262.255 119.38 0)
+      (effects (font (size 1.27 1.27)) hide)
+    )
+    (pin "1")
+  )
   (symbol (lib_id "power:+5V") (at 135.89 49.53 0) (unit 1)

Commit message: change the file name debugger-code into debugger_code_f103. Change the stm32f103rct6 into stm32f407vet6. Add file debugger_code_f407
Parts:
- added H1: mountinghole, MountingHole:MountingHole_2.1mm, symbol 301_Link_Pad:mountinghole
- added J5: Conn_01x02, Connector_JST:JST_GH_SM02B-GHS-TB_1x02-1MP_P1.25mm_Horizontal, symbol Connector_Generic:Conn_01x02
- renumbered C8 to C10, C4 to C11, C5 to C2, C6 to C3, C2 to C4, C9 to C5, C3 to C6, C10 to C8, C11 to C9, J4 to J2, J2 to J3, J3 to J4, R10 to R2, R2 to R3, R11 to R4, U3 to U2, U2 to U3
Connections:
- net +5V: now also J5.2 (Pin_2)
- net GND: now also J5.1 (Pin_1)

Commit message: temp.change the PCB.And change the code.
Parts:
- removed C1, C4, C6: 10u, Capacitor_SMD:C_0603_1608Metric, symbol Device:C_Small
- removed C2, C3, C7: 100n, Capacitor_SMD:C_0603_1608Metric, symbol Device:C_Small
- removed D1: LED, LED_SMD:LED_0603_1608Metric, symbol Device:LED
- removed H1: mountinghole, MountingHole:MountingHole_2.1mm, symbol 301_Link_Pad:mountinghole
- removed J5: Conn_01x02, Connector_JST:JST_GH_SM02B-GHS-TB_1x02-1MP_P1.25mm_Horizontal, symbol Connector_Generic:Conn_01x02
- removed R1: 1k, Resistor_SMD:R_0603_1608Metric, symbol Device:R_Small
- removed R4: 10k, Resistor_SMD:R_0603_1608Metric, symbol Device:R_Small
- removed U1, U3: HX9193, Package_TO_SOT_SMD:SOT-23-5_HandSoldering, symbol symbol:HX9193
- added C10: 101, Capacitor_SMD:C_0603_1608Metric, symbol Device:C
- added C11, C12, C13, C15: 22u, Capacitor_SMD:C_1206_3216Metric, symbol Basic_passive_components:Capacitor
- added C12: 100n, Capacitor_SMD:C_0805_2012Metric, symbol Device:C_Small
- added C13, C8: 100n, Capacitor_SMD:C_0603_1608Metric, symbol Device:C
- added C25, C27, C9: 4.7u, Capacitor_SMD:C_0603_1608Metric, symbol Device:C_Small
- added C26, C28: 100n, Capacitor_SMD:C_0603_1608Metric, symbol Device:C_Small
- added C42: 104, Capacitor_SMD:C_0603_1608Metric, symbol Device:C
- added C5: 103, Capacitor_SMD:C_0603_1608Metric, symbol Device:C
- added C6: 22uf 0603, Capacitor_SMD:C_1206_3216Metric, symbol Device:C
- added C7: 100n, Capacitor_SMD:C_0603_1608Metric, symbol Basic_passive_components:Capacitor
- added C8: 10u, Capacitor_SMD:C_1206_3216Metric, symbol Basic_passive_components:Capacitor
- added C9: 106 1206, Capacitor_SMD:C_1206_3216Metric, symbol Device:C
- added D1, D2, D3, D4, D6: (no value), LED_SMD:LED_0603_1608Metric, symbol Basic_semiconductor:Diode_LED
- added D1 (x2): LED, LED_SMD:LED_0603_1608Metric, symbol Device:LED
- added H8, H9: MountingHole, ic:mo, symbol Mechanical:MountingHole
- added J1: axt430124, Connector_PinHeader_1.27mm:PinHeader_2x15_P1.27mm_Vertical, symbol Connector_Generic:Conn_02x15_Odd_Even
- added J1: Conn_01x14, Connector_FFC-FPC:Hirose_FH12-14S-0.5SH_1x14-1MP_P0.50mm_Horizontal, symbol Connector_Generic:Conn_01x14
- added J5, J9: Conn_01x02, Connector_PinHeader_2.54mm:PinHeader_1x02_P2.54mm_Vertical, symbol 302_Link_W2B-Connector:Conn_01x02
- added J8: USB_C_Receptacle_USB2.0, Connector_USB:USB_C_Receptacle_HRO_TYPE-C-31-M-12, symbol Connector:USB_C_Receptacle_USB2.0
- added L1: 1u, PCM_008_GN_POWER-CHOKE_SMD:MC-0630, symbol Device:L
- added L1: 600r, Inductor_SMD:L_0805_2012Metric, symbol Device:L
- added L1: 2.2uh, Inductor_SMD_Wurth:L_Wurth_WE-LQSH-4020, symbol Device:L
- added Q1: SI2301, Package_TO_SOT_SMD:SOT-23, symbol Device:Q_PMOS_GSD
- added Q3: AO3407, Package_TO_SOT_SMD:SOT-23, symbol Device:Q_PMOS_GSD
- added R1: 200K, Resistor_SMD:R_0603_1608Metric, symbol Device:R
- added R15: 10k, Resistor_SMD:R_0603_1608Metric, symbol Device:R
- added R15, R16, R17, R18, R22, R23: 10k, Resistor_SMD:R_0603_1608Metric, symbol Basic_passive_components:Resistor
- added R3 (x2): 1K, Resistor_SMD:R_0603_1608Metric, symbol Device:R_Small
- added R3: 220K, Resistor_SMD:R_0603_1608Metric, symbol Device:R
- added R4: 30k, Resistor_SMD:R_0603_1608Metric, symbol Device:R
- added SW1: SW_SPDT, Button_Switch_SMD:SW_SPDT_PCM12, symbol Switch:SW_SPDT
- added U1, U8: ~, Package_DFN_QFN:DFN-8-1EP_3x3mm_P0.65mm_EP1.55x2.4mm, symbol ldo:AP7361C
- added U1: SY8303, PCM_003_GN_SMALL-SEMI_SMD:SOT-23-8, symbol PCM_204_Power_SMPS-Convertor:SY8303
- added U3: IP5306, PCM_004_GN_MIDDLE-SEMI_SMD:SOP-8EP_3949, symbol Armor:IP5306
- added U5: pesd1can, PCM_003_GN_SMALL-SEMI_SMD:SOT-23, symbol 103_IntegratedCircuit_Reference:REF3030
- C11: value 10u -> 4.7u; footprint Capacitor_SMD:C_0603_1608Metric -> Capacitor_SMD:C_0805_2012Metric
- R2: value 10k -> 10K
Connections:
- net +5V: now also C10.2, C10.2, C11.1, C12.1, C13.1, C15.1, C25.2, C26.2, C42.2, C6.2, C9.2, J1.2 (Pin_2), L1.2, R3.2, U1.5 (EN), U1.8 (IN), U3.8 (VOUT), U8.5 (EN), U8.8 (IN)
- net CAN+: now also U5.1 (Vin); no longer R2.2
- net CAN-: now also U5.2 (Vout)
- net GND: now also C10.1, C11.1, R2.2, C12.1, C13.2, C25.1, C26.1, C27.1, C28.1, C42.1, C6.1, C7.1, C8.1, C8.1, C9.1, C9.1, D1.1 (K), D1.1 (K), D6.1 (Cathode), J1.1 (Pin_1), J1.28 (Pin_28), J1.29 (Pin_29), J1.30 (Pin_30), J5.1, J8.A1 (GND), J8.A12 (GND), J8.B1 (GND), J8.B12 (GND), J8.S1 (SHIELD), R1.2, R23.1, R4.1, SW1.3 (C), U1.3 (GND), U1.4 (GND), U1.4 (GND), U1.9 (GND), U3.EP (GND), U5.3 (GND), U8.4 (GND), U8.9 (GND); no longer C10.2, C11.2, R2.1
- net LCD_3V3: now also C11.2, C12.2, J1.1 (Pin_1), Q1.2 (S), U1.1 (OUT); no longer C10.1, C11.1
- net VCC: now also C27.2, C28.2, J9.2, L1.1, R3.1, R3.1, U8.1 (OUT)
- new net: D6.2 (Anode), R22.1
- new net: D4.1 (Cathode), R18.1
- new net: D1.1 (Cathode), D2.2 (Anode), D3.1 (Cathode), D4.2 (Anode), U3.4 (LED3)
- new net: D1.2 (A), R3.2 (x2)
- new net: R15.2, R16.2, U3.2 (LED1)
- new net: R17.2, R18.2, U3.3 (LED2)
- new net: R22.2, R23.2, U3.5 (KEY)
- new net: L1.1, U3.7 (SW)
- new net: J1.2 (Pin_2), Q1.3 (D)
- new net: D1.2 (Anode), R15.1
- new net: C10.1, R3.1, R4.2, U1.1 (FB)
- new net: C5.1, U1.7 (BST)
- new net: C5.2, L1.1, U1.6 (SW)
- new net: R1.1, U1.2 (FS)
- new net: C8.2, C9.2, L1.2, U1.5 (VIN), U1.8 (EN)
- new net: D3.2 (Anode), R17.1
- new net: D2.1 (Cathode), R16.1
- new net ADC1_IN0: J1.12 (Pin_12)
- new net ADC1_IN1: J1.14 (Pin_14)
- new net ADC1_IN11: J1.4 (Pin_4)
- new net ADC1_IN12: J1.6 (Pin_6)
- new net ADC1_IN13: J1.8 (Pin_8)
- new net ADC1_IN14: J1.10 (Pin_10)
- new net BATE_5V: C7.2, C8.2, J8.A4 (VBUS), J8.A9 (VBUS), J8.B4 (VBUS), J8.B9 (VBUS), U3.1 (VIN)
- new net G: C13.1, Q3.1 (G), R15.1, SW1.1 (A), SW1.2 (B)
- new net GND1: C11.2, C12.2, C13.2, C15.2, J9.1
- new net I2C3_SCL: J1.27 (Pin_27)
- new net I2C3_SDA: J1.25 (Pin_25)
- new net KEY1: J1.8 (Pin_8)
- new net KEY2: J1.9 (Pin_9)
- new net KEY3: J1.10 (Pin_10)
- new net KEY4: J1.11 (Pin_11)
- new net KEY5: J1.12 (Pin_12)
- new net LCD_A0: J1.5 (Pin_5)
- new net LCD_CLK: J1.3 (Pin_3), J1.9 (Pin_9)
- new net LCD_CS: J1.11 (Pin_11)
- new net LCD_CS0: J1.7 (Pin_7)
- new net LCD_DC: J1.6 (Pin_6)
- new net LCD_LED: J1.13 (Pin_13), Q1.1 (G), R2.1
- new net LCD_MOSI: J1.4 (Pin_4), J1.7 (Pin_7)
- new net LCD_RST: J1.3 (Pin_3), J1.5 (Pin_5)
- new net RESET: J1.14 (Pin_14)
- new net TIM1_CH1: J1.26 (Pin_26)
- new net TIM1_CH2: J1.24 (Pin_24)
- new net TIM3_CH1: J1.16 (Pin_16)
- new net TIM3_CH2: J1.18 (Pin_18)
- new net TIM4_CH1: J1.20 (Pin_20)
- new net TIM4_CH2: J1.22 (Pin_22)
- new net TOUCH_CLK: J1.15 (Pin_15)
- new net TOUCH_CS: J1.23 (Pin_23)
- new net TOUCH_INT: J1.21 (Pin_21)
- new net TOUCH_MISO: J1.17 (Pin_17)
- new net TOUCH_MOSI: J1.19 (Pin_19)
- new net VBAT: L1.2, Q3.3 (D), U3.6 (BAT)
- new net VBAT+: J5.2, Q3.2 (S), R15.2
- no-connect marks 7 -> 14
Other:
- note added: "PWR"
- moved on the sheet: C5, C8, C9, J1, J2, J3, J4, R3, U2, U4
